Commit message: Update rosbob_v3.xacro

File: shared_tavern/urdf/rosbob_v3.xacro (robot description, xacro)
@@ -142,5 +142,5 @@
 	<link name="robot_footprint"></link>
 	<!-- Camera -->
-	<link name="camera">
+	<!-- <link name="camera">
 		<inertial>
 			<mass value="${camera_mass}"/>
@@ -164,7 +164,7 @@
 			</geometry>
 		</collision>
-	</link>
+	</link> -->
 	<!-- Hokuyo Lidar -->
-	<link name="hokuyo">
+	<!-- <link name="hokuyo">
 		<inertial>
 			<mass value="${hokoyu_mass}"/>
@@ -188,5 +188,5 @@
 			</geometry>
 		</collision>
-	</link>
+	</link> -->
 		<!-- Define Joints -->
 	<!-- Right Wheel Joint Back-->
@@ -237,20 +237,34 @@
 	</joint>
 	<!-- Camera Joint -->
-	<joint name="camera_joint" type="fixed">
+	<!-- <joint name="camera_joint" type="fixed">
 		<origin xyz="0.25 0.1 0.4529" rpy="0 0 0" />
 		<parent link="base_link"/>
 		<child link="camera" />
 		<axis xyz="0 1 0"/>
-	</joint>
+	</joint> -->
 	<!-- Hokoyu Joint -->
-	<joint name="hokuyo_joint" type="fixed">
+	<!-- <joint name="hokuyo_joint" type="fixed">
 	    <origin xyz="0.3 0 0.4629" rpy="0 0 0" />
 	    <parent link="base_link"/>
 	    <child link="hokuyo" />
 	    <axis xyz="0 1 0"/>
-	</joint>
+	</joint> -->
+	<!-- JOIN ARM URDF !!!!!!!!!!!!!!!!!!-->
+	<joint name="arm_fixed_joint" type="fixed">
+      <parent link="base_link" />
+      <child link = "arm_link" />
+      <origin xyz="0.0 0.0 0.0" rpy="0.0 0.0 0.0" />
+    </joint>
+    <link name="arm_link">
+      <collision>
+        <geometry>
+          <box size="0.01 0.01 0.01"/>
+        </geometry>
+        <origin rpy="0 0 0" xyz="0 0 0"/>
+      </collision>
+    </link>
 	<!-- Color of bot -->
 	<gazebo reference="left_wheel_front">
-		<material>Gazebo/Green</material>
+		<material>Gazebo/Grey</material>
 		<kp>1000000.0</kp> <!-- kp and kd for rubber -->
 		<kd>100.0</kd>
@@ -261,5 +275,5 @@
 	</gazebo>
 	<gazebo reference="left_wheel_back">
-		<material>Gazebo/Blue</material>
+		<material>Gazebo/Grey</material>
 		<kp>1000000.0</kp> <!-- kp and kd for rubber -->
 		<kd>100.0</kd>
@@ -270,5 +284,5 @@
 	</gazebo>
 	<gazebo reference="right_wheel_front">
-		<material>Gazebo/Red</material>
+		<material>Gazebo/Grey</material>
 		<kp>1000000.0</kp> <!-- kp and kd for rubber -->
 		<kd>100.0</kd>
@@ -279,5 +293,5 @@
 	</gazebo>
 	<gazebo reference="right_wheel_back">
-		<material>Gazebo/Yellow</material>
+		<material>Gazebo/Grey</material>
 		<kp>1000000.0</kp> <!-- kp and kd for rubber -->
 		<kd>100.0</kd>
